File: expansions/extra_av_out/extra_av_out.kicad_sch (KiCad schematic)
At the start: 53 parts, among them J1 Conn_02x25_Odd_Even, J2 SJ1-3533NG, J3 PLT133/T10W, J4 VGA, Q1 BC847, U1 ADV7125KSTZ140, U2 PCM5142PW, U3 74HCT2G17GW

Commit message: update extra_av_out to v1.2
* fix Toslink footprint pin order
Parts:
- J3: footprint custom_components:EAPLRAA4 -> custom_components:PLT133
Connections:
- no-connect marks 16 -> 18
Changed lines of the file:
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@@
   (title_block
     (title "Extra AV out board")
-    (date "2023-12-11")
-    (rev "1.1")
+    (date "2024-04-05")
+    (rev "1.2")
   )
   (junction (at 43.18 151.13) (diameter 0) (color 0 0 0 0)
@@
   (no_connect (at 26.67 54.61))
   (no_connect (at 26.67 105.41))
+  (no_connect (at 247.65 154.94))
   (no_connect (at 26.67 57.15))
   (no_connect (at 143.51 158.75))
@@
   (no_connect (at 256.54 90.17))
   (no_connect (at 256.54 95.25))
+  (no_connect (at 247.65 157.48))
   (no_connect (at 143.51 153.67))
   (no_connect (at 39.37 57.15))
@@
       (effects (font (size 1.27 1.27)) (justify right))
     )
-    (property "Footprint" "custom_components:EAPLRAA4" (at 240.03 35.56 0)
-      (effects (font (size 1.27 1.27)) hide)
-    )
+    (property "Footprint" "custom_components:PLT133" (at 240.03 35.56 0)
+      (effects (font (size 1.27 1.27)) hide)
+    )
