File: afe_rgb.kicad_sch (KiCad schematic)
At the start: 55 parts, among them U8 ISL51002CQZ-165

Commit message: update schematic to v1.5
Connections:
- net ISL_CLAMP is gone; now on net GND: U8.63 (CLAMPIN)
- net ISL_COAST is gone; now on net GND: U8.64 (COASTIN)

Commit message: update schematic to v1.6
Parts:
- removed C41, C42, C43, C44: 50p, Capacitor_SMD:C_0402_1005Metric, symbol Device:C_Small
- removed R22, R24, R26, R27: 1k, Resistor_SMD:R_0402_1005Metric, symbol Device:R_Small
- removed R23, R25, R28, R29: 1.9k, Resistor_SMD:R_0402_1005Metric, symbol Device:R_Small
- added C333, C334: 0.1u, Capacitor_SMD:C_0402_1005Metric, symbol Device:C_Small
- added U32, U33: SN74LVC2G17, Package_TO_SOT_SMD:SC-70-8, symbol custom_components:SN74LVC2G17
Connections:
- net AV1_HS: now also U33.1 (1A)
- net AV1_HS_3v3: now also U33.6 (1Y)
- net AV1_VS: now also U33.3 (2A)
- net AV1_VS_3v3: now also U33.4 (2Y)
- net AV3_HS: now also U32.1 (1A)
- net AV3_HS_3v3: now also U32.6 (1Y)
- net AV3_VS: now also U32.3 (2A)
- net AV3_VS_3v3: now also U32.4 (2Y)
- net DVDD3v3: now also C333.1, C334.1, U32.5 (Vcc), U33.5 (Vcc)
- net GND: now also C333.2, C334.2, U32.2 (GND), U33.2 (GND)
