File: fpga2.kicad_sch (KiCad schematic)
At the start: 4 parts, among them P1 5CEFA7F23

Commit message: update schematic to v1.5
Parts:
- P1: value 5CEFA7F23 -> 5CEFA5F23
Connections:
- net BTN2: now also P1.U17 (IO_4A)
- net BTN3: now also P1.U20 (IO_4A)
- net EXP_IO_A_2: now also P1.V21 (IO_4A)
- net EXP_IO_A_3: now also P1.V18 (IO_4A)
- net EXP_IO_A_4: now also P1.U16 (IO_4A)
- net EXP_IO_A_5: now also P1.U21 (IO_4A)
- net HDMIRX_B0: now also P1.V13 (IO_4A)
- net HDMIRX_B1: now also P1.AB12 (IO_4A)
- net HDMIRX_B2: now also P1.U13 (IO_4A)
- net HDMIRX_B3: now also P1.T12 (IO_4A)
- net HDMIRX_B4: now also P1.AA14 (IO_4A)
- net HDMIRX_B5: now also P1.T13 (IO_4A)
- net HDMIRX_B6: now also P1.AA13 (IO_4A)
- net HDMIRX_B7: now also P1.AB15 (IO_4A)
- net HDMIRX_DE: now also P1.AA22 (IO_4A)
- net HDMIRX_G0: now also P1.Y14 (IO_4A)
- net HDMIRX_G1: now also P1.AA15 (IO_4A)
- net HDMIRX_G2: now also P1.Y15 (IO_4A)
- net HDMIRX_G3: now also P1.AB17 (IO_4A)
- net HDMIRX_G4: now also P1.AB18 (IO_4A)
- net HDMIRX_G5: now also P1.AB20 (IO_4A)
- net HDMIRX_G6: now also P1.Y16 (IO_4A)
- net HDMIRX_G7: now also P1.AB21 (IO_4A)
- net HDMIRX_HSYNC: now also P1.W19 (IO_4A)
- net HDMIRX_I2S0: now also P1.Y20 (IO_4A)
- net HDMIRX_I2S_BCK: now also P1.Y19 (IO_4A)
- net HDMIRX_I2S_WS: now also P1.W22 (IO_4A)
- net HDMIRX_R0: now also P1.Y17 (IO_4A)
- net HDMIRX_R1: now also P1.T14 (IO_4A)
- net HDMIRX_R2: now also P1.AA17 (IO_4A)
- net HDMIRX_R3: now also P1.U15 (IO_4A)
- net HDMIRX_R4: now also P1.AA18 (IO_4A)
- net HDMIRX_R5: now also P1.AA19 (IO_4A)
- net HDMIRX_R6: now also P1.V20 (IO_4A)
- net HDMIRX_R7: now also P1.AA20 (IO_4A)
- net HDMIRX_VSYNC: now also P1.AB22 (IO_4A)
- net HDMITX_5V_EN: now also P1.L22 (IO_5B)
- net HDMITX_B4: now also P1.K22 (IO_5B)
- net HDMITX_B5: now also P1.L18 (IO_5B)
- net HDMITX_B6: now also P1.K21 (IO_5B)
- net HDMITX_B7: now also P1.L19 (IO_5B)
- net HDMITX_G0: now also P1.M21 (IO_5B)
- net HDMITX_G1: now also P1.L17 (IO_5B)
- net HDMITX_G2: now also P1.M20 (IO_5B)
- net HDMITX_G3: now also P1.K17 (IO_5B)
- net HDMITX_G4: now also P1.M18 (IO_5B)
- net HDMITX_G5: now also P1.N19 (IO_5B)
- net HDMITX_G6: now also P1.N21 (IO_5B)
- net HDMITX_G7: now also P1.N20 (IO_5B)
- net HDMITX_I2S0: now also P1.R14 (IO_4A)
- net HDMITX_I2S_BCK: now also P1.U22 (IO_4A)
- net HDMITX_I2S_WS: now also P1.W21 (IO_4A)
- net HDMITX_PCLK: now also P1.M22 (IO_5B)
- net HDMITX_R0: now also P1.P17 (IO_5A)
- net HDMITX_R1: now also P1.P18 (IO_5A)
- net HDMITX_R2: now also P1.P16 (IO_5A)
- net HDMITX_R3: now also P1.P19 (IO_5A)
- net HDMITX_R4: now also P1.R17 (IO_5A)
- net HDMITX_R5: now also P1.R16 (IO_5A)
- net HDMITX_R6: now also P1.R15 (IO_5A)
- net HDMITX_R7: now also P1.T15 (IO_5A)
- net HDMITX_SPDIF: now also P1.V19 (IO_4A)
- net HDMI_RESET#: now also P1.Y22 (IO_4A)
- net SCL: now also P1.P14 (IO_4A)
- net SDA: now also P1.Y21 (IO_4A)
