File: io_digital_av.kicad_sch (KiCad schematic)
At the start: 27 parts, among them J12 EAPLRAA4, J2 10029449-111RLF, J3 10029449-111RLF, Q7 AOSS21115C, Q8 BC847

Commit message: update schematic to v1.5
Parts:
- J12: value EAPLRAA4 -> FCR684208R; footprint custom_components:EAPLRAA4 -> custom_components:FCR684208R

Commit message: fix power supply connections on v1.6 schematic
Changed lines of the file:
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@@
 (kicad_sch
-	(version 20231120)
+	(version 20250114)
 	(generator "eeschema")
-	(generator_version "8.0")
+	(generator_version "9.0")
 	(paper "A4")
 	(title_block
@@
 	(label "HDMIRX_DDC5V"
 		(at 26.67 143.51 0)
-		(fields_autoplaced yes)
 		(effects
 			(font
@@
 	(label "HDMIRX_CEC"
 		(at 135.89 151.13 0)
-		(fields_autoplaced yes)
 		(effects
 			(font
@@
 	(label "HDMITX_DDCSCL"
 		(at 134.62 78.74 0)
-		(fields_autoplaced yes)
 		(effects
 			(font
@@
 	(label "HDMIRX_DDCSDA"
 		(at 135.89 158.75 0)
-		(fields_autoplaced yes)
 		(effects
 			(font
@@
 	(label "HDMITX_HPD"
 		(at 134.62 76.2 0)
-		(fields_autoplaced yes)
 		(effects
 			(font
@@
 	(label "HDMIRX_HPA"
 		(at 135.89 153.67 0)
-		(fields_autoplaced yes)
 		(effects
 			(font
@@
 	(label "HDMIRX_DDCSCL"
 		(at 135.89 156.21 0)
-		(fields_autoplaced yes)
 		(effects
 			(font
@@
 	(label "HDMITX_CEC"
 		(at 137.16 62.23 0)
-		(fields_autoplaced yes)
 		(effects
 			(font
@@
 	(label "HDMIRX_CEC"
 		(at 138.43 139.7 0)
-		(fields_autoplaced yes)
 		(effects
 			(font
@@
 	(label "HDMITX_DDCSDA"
 		(at 134.62 81.28 0)
-		(fields_autoplaced yes)
 		(effects
 			(font
@@
 	(label "HDMITX_CEC"
 		(at 134.62 73.66 0)
-		(fields_autoplaced yes)
 		(effects
 			(font
