File: memory.kicad_sch (KiCad schematic)
At the start: 51 parts, among them U10 N25Q128A13ESE40G, U9 MT42L64M32D2HE-18 AAT:D

Commit message: update schematic to v1.5
Parts:
- U9: value MT42L64M32D2HE-18 AAT:D -> MT42L32M32D1HE-18 IT:D
Connections:
- net DVDD1v2: now also U9.B5 (VDD2), U9.C10 (VDDQ), U9.C7 (VDDQ), U9.D2 (VDD2), U9.D5 (VDDQ), U9.E9 (VDDQ), U9.F1 (VDDCA), U9.F10 (VDDQ), U9.G1 (VDD2), U9.H1 (VDDCA), U9.H6 (VDDQ), U9.J6 (VDDQ), U9.J7 (VDD2), U9.K6 (VDDQ), U9.M10 (VDDQ), U9.N2 (VDDCA), U9.N9 (VDDQ), U9.P2 (VDD2), U9.P5 (VDDQ), U9.R10 (VDDQ), U9.R7 (VDDQ), U9.T5 (VDD2)
- net DVDD1v8: now also U9.B6 (VDD1), U9.C1 (VDD1), U9.R1 (VDD1), U9.T6 (VDD1)
- net GND: now also U9.C2 (VSS), U9.C5 (VSS), U9.C6 (VSSQ), U9.C9 (VSSQ), U9.D1 (VSS), U9.D10 (VSSQ), U9.E1 (VSSCA), U9.E10 (VSSQ), U9.F5 (VSSQ), U9.G10 (VSSQ), U9.H2 (VSS), U9.J1 (VSSCA), U9.J5 (VSSQ), U9.J8 (VSS), U9.L10 (VSSQ), U9.M5 (VSSQ), U9.N1 (VSSCA), U9.N10 (VSSQ), U9.P1 (VSS), U9.P10 (VSSQ), U9.R2 (VSS), U9.R5 (VSS), U9.R6 (VSSQ), U9.R9 (VSSQ)
- net VREFCA_LPDDR2: now also U9.G3 (VREFCA)
- net VREFDQ_LPDDR2: now also U9.J9 (VREFDQ)
- net at R78.1: now also U9.D3 (ZQ0)
- net at R77.1: now also U9.C3 (ZQ1)
